File: Boards/Baseboard/Baseboard.kicad_pcb (KiCad board)
At the start: 2 copper layers, 160 x 50 mm, 46 parts, among them CON1 BARREL_JACK, IC1 MC34063AP, IC2 74HCT245DW, J1 Serial, J2 Display, P1 HV_Supply, Q1 IRF740, Q2 MPSA55, Q3 BC327, Q4 BC337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

Commit message: Layout chnages
Parts:
- removed P1: HV_Supply, Socket_Strips:Socket_Strip_Straight_1x03_Pitch2.54mm
- added J3: HV, Socket_Strips:Socket_Strip_Straight_1x02_Pitch2.54mm, F.Cu at (237.4, 87.3)
- added R11: 1R, Resistors_THT:R_Axial_DIN0207_L6.3mm_D2.5mm_P10.16mm_Horizontal, F.Cu at (179.8, 65.5)
- added R15: 1R, Resistors_THT:R_Axial_DIN0207_L6.3mm_D2.5mm_P10.16mm_Horizontal, F.Cu at (192.0, 65.5)
- added R16: 1R, Resistors_THT:R_Axial_DIN0207_L6.3mm_D2.5mm_P10.16mm_Horizontal, F.Cu at (188.0, 65.5)
- D4: value Time -> Status
- Q3, Q4: footprint TO_SOT_Packages_THT:TO-92_Molded_Narrow -> TO_SOT_Packages_THT:TO-92_Inline_Wide
- R12: value 475k -> 470k
- R13: value 475k -> 1k
- R2: value 0R33 -> 1R
- R4: value 3k32 -> 3k4
- moved R2 45.7 mm to (183.9, 65.5), turned to 270 degrees
- moved R14 11.7 mm to (180.3, 80.6)
- moved Q4 8.64 mm to (183.5, 85.1)
- moved C12 4.34 mm to (100.6, 79.8), turned to 0 degrees
- moved J2 2.25 mm to (87.4, 79.7)
- moved C1 1.91 mm to (216.7, 98.0)
- moved C3 1.91 mm to (202.7, 98.0)
- moved C4 1.91 mm to (202.1, 82.8)
- moved C5 1.91 mm to (195.7, 94.3)
- moved D1 1.91 mm to (220.5, 73.3)
- moved D2 1.91 mm to (216.7, 73.3)
- moved IC1 1.91 mm to (208.1, 86.8)
- moved L1 1.91 mm to (216.7, 90.7)
- moved Q1 1.91 mm to (226.1, 96.0)
- moved Q2 1.91 mm to (212.9, 83.4)
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Connections:
- net HV_EN renamed HV_Off
- net Net-(C2-Pad1) renamed /175V
Routing:
- net Net-(C1-Pad1): track 34.6 -> 95.0 mm
- net Net-(Q4-Pad1): track 11.2 -> 23.5 mm
- net +12V: track 118.9 -> 130.1 mm, vias 0 -> 1
- net Net-(D1-Pad2): track 40.8 -> 29.9 mm
- net Net-(Q4-Pad2): track 5.08 -> 9.05 mm
- net /175V: track 60.6 -> 63.5 mm
- net +5V: track 118.2 -> 115.7 mm, vias 1 -> 2
- net GND: track 44.5 -> 46.3 mm, vias 6 -> 5
- net Net-(C5-Pad1): track 17.3 -> 15.5 mm
- net Net-(IC2-Pad4): track 8.60 -> 7.08 mm
- net HV_Off: track 56.8 -> 58.3 mm, vias 1 -> 2
- net Net-(IC2-Pad2): track 10.3 -> 11.6 mm
- net Net-(Q3-Pad2): track 11.8 -> 13.0 mm
- net Net-(IC2-Pad5): track 6.38 -> 6.92 mm

Commit message: Board layout done
Parts:
- added C13: 100nF, Capacitors_SMD:C_0805_HandSoldering, F.Cu at (117.5, 99.1)
- added C14: 1.5nF, Capacitors_THT:C_Disc_D3.0mm_W2.0mm_P2.50mm, F.Cu at (201.9, 67.3)
- added D5: LED, LEDs:LED_D3.0mm, F.Cu at (184.2, 74.3)
- added D6: D_TVS, Diodes_THT:D_5W_P12.70mm_Horizontal, F.Cu at (167.6, 80.6)
- added D7: 1N5711, Diodes_THT:D_DO-35_SOD27_P10.16mm_Horizontal, F.Cu at (199.4, 87.6)
- added D8: ZD20 / 1W, Diodes_THT:D_DO-41_SOD81_P10.16mm_Horizontal, F.Cu at (217.2, 83.2)
- added J4: Sensor, Measurement_Points:Measurement_Point_Square-TH_Small, F.Cu at (108.6, 106.0)
- added Q5: BS170, TO_SOT_Packages_THT:TO-92_Molded_Narrow, F.Cu at (194.3, 69.8)
- added Q6: BC337, TO_SOT_Packages_THT:TO-92_Inline_Wide, F.Cu at (194.9, 89.5)
- added Q7: MPSA42, TO_SOT_Packages_THT:TO-92_Molded_Narrow, F.Cu at (201.3, 73.0)
- added Q8: BC337, TO_SOT_Packages_THT:TO-92_Inline_Wide, F.Cu at (201.3, 81.3)
- added R17: 220k, Resistors_THT:R_Axial_DIN0207_L6.3mm_D2.5mm_P10.16mm_Horizontal, F.Cu at (221.0, 73.0)
- added R18: 120k, Resistors_THT:R_Axial_DIN0207_L6.3mm_D2.5mm_P10.16mm_Horizontal, F.Cu at (210.8, 65.4)
- added R19: 680R, Resistors_THT:R_Axial_DIN0207_L6.3mm_D2.5mm_P10.16mm_Horizontal, F.Cu at (188.6, 74.3)
- added R20: 10k, Resistors_SMD:R_0805_HandSoldering, F.Cu at (113.0, 97.8)
- added R21: 10k, Resistors_SMD:R_0805_HandSoldering, F.Cu at (121.3, 99.1)
- added R22: 1k, Resistors_THT:R_Axial_DIN0207_L6.3mm_D2.5mm_P10.16mm_Horizontal, F.Cu at (192.4, 87.0)
- added R23: 47R, Resistors_THT:R_Axial_DIN0207_L6.3mm_D2.5mm_P10.16mm_Horizontal, F.Cu at (210.8, 69.2)
- added R24: 4k7, Resistors_THT:R_Axial_DIN0207_L6.3mm_D2.5mm_P10.16mm_Horizontal, F.Cu at (196.2, 87.0)
- added R26: 1k, Resistors_THT:R_Axial_DIN0207_L6.3mm_D2.5mm_P10.16mm_Horizontal, F.Cu at (181.0, 81.3)
- added REF**: Symbol_HighVoltage_Type2_CopperTop_VerySmall, MySymbols:Symbol_HighVoltage_Type2_SilkTop_VerySmall, F.Cu at (176.8, 69.6)
- added RV1: 100k, Potentiometers:Potentiometer_Trimmer_Piher_PT-6h_Vertical, F.Cu at (99.7, 99.7)
- added RV2: 500R, Potentiometers:Potentiometer_Trimmer_Bourns_PV36W, F.Cu at (190.5, 103.5)
- added U4: MTCH101, TO_SOT_Packages_SMD:SOT-23-6_Handsoldering, F.Cu at (113.0, 101.0)
- C4: value 2µ2 -> 1.5nF; footprint Capacitors_THT:CP_Radial_D6.3mm_P2.50mm -> Capacitors_THT:C_Disc_D3.0mm_W2.0mm_P2.50mm
- C5: value 100nF -> 10nF
- D1: value BAV21 -> MUR120; footprint Diodes_THT:D_DO-35_SOD27_P10.16mm_Horizontal -> Diodes_THT:D_DO-15_P10.16mm_Horizontal
- L1: value 220µH -> 270µH / 1.2A; footprint Inductors_THT:L_Radial_D6.0mm_P4.00mm -> Inductors_THT:L_Radial_D12.5mm_P7.00mm_Fastron_09HCP
- Q2: value MPSA55 -> BC327
- R1: value 475k -> 549k
- R10, R5: value R -> 68R
- R12: value 470k -> 4k7
- R13: value 1k -> 180R
- R14: value 4k7 -> 1k
- R4: value 3k4 -> 3k3
- R8: value 470R -> 10k
- moved R15 40.8 mm to (181.0, 104.8), turned to 90 degrees
- moved R16 40.7 mm to (177.2, 104.8), turned to 90 degrees
- moved R2 40.6 mm to (173.4, 104.8), turned to 90 degrees
- moved R11 40.6 mm to (169.5, 104.8), turned to 90 degrees
- moved R1 37.6 mm to (232.4, 98.4)
- moved C2 35.0 mm to (227.3, 103.5), turned to 270 degrees
- moved R8 29.1 mm to (103.5, 102.2), turned to 180 degrees
- moved R13 27.6 mm to (208.3, 104.1), turned to 180 degrees
- moved D1 26.1 mm to (227.3, 98.4), turned to 90 degrees
- moved Q3 22.6 mm to (206.4, 76.8), turned to 90 degrees
- moved R9 17.5 mm to (129.5, 69.8), turned to 180 degrees
- moved R4 15.6 mm to (184.8, 94.6)
- moved R10 15.4 mm to (129.5, 103.5), turned to 180 degrees
- moved D4 15.4 mm to (129.5, 106.0), turned to 180 degrees
- moved R6 11.7 mm to (99.7, 69.8)
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Connections:
- net HV_Off renamed HV_On
- IC1 pad 3: Net-(C4-Pad1) -> Net-(D7-Pad2)
- IC1 pad 8: Net-(C1-Pad1) -> Net-(IC1-Pad8)
- Q2 pad 1: Net-(D2-Pad2) -> GND
- Q2 pad 2: GND -> Net-(D7-Pad2)
- Q2 pad 3: Net-(D2-Pad1) -> Net-(C4-Pad1)
- Q3 pad 1: Net-(C5-Pad1) -> GND
- Q3 pad 2: Net-(Q3-Pad2) -> Net-(D2-Pad2)
- Q3 pad 3: +12V -> Net-(D2-Pad1)
- R12 pad 1: Net-(Q3-Pad2) -> Net-(Q4-Pad1)
- R13 pad 1: Net-(Q4-Pad1) -> Net-(IC1-Pad8)
- R13 pad 2: Net-(Q3-Pad2) -> Net-(C1-Pad1)
- R4 pad 2: Net-(C5-Pad1) -> Net-(R4-Pad2)
- R8 pad 2: GND -> Net-(R8-Pad2)
- U2 pad 11: Net-(R8-Pad1) -> Net-(R10-Pad1)
- U2 pad 13: Net-(R10-Pad1) -> Prx_Det
Routing:
- net GND: track 46.3 -> 110.5 mm, vias 5 -> 27
- net Net-(Q5-Pad2): track 0.00 -> 42.5 mm
- net Net-(C5-Pad1): track 15.5 -> 57.7 mm
- net Net-(C14-Pad2): track 0.00 -> 28.9 mm
- net Prx_Det: track 0.00 -> 27.3 mm, vias 0 -> 2
- net Net-(Q8-Pad2): track 0.00 -> 22.0 mm
- net Net-(R9-Pad1): track 3.77 -> 23.0 mm
- net Net-(R9-Pad2): track 25.0 -> 6.40 mm
- net /175V: track 63.5 -> 46.7 mm
- net Net-(D1-Pad2): track 29.9 -> 13.2 mm
- net Net-(D7-Pad2): track 0.00 -> 16.1 mm
- net +3V3: track 73.5 -> 88.7 mm, vias 4 -> 7
- net Net-(Q4-Pad1): track 23.5 -> 9.20 mm
- net Net-(R6-Pad1): track 3.67 -> 17.6 mm
- net Net-(C14-Pad1): track 0.00 -> 13.5 mm
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Other:
- board text added: "+"
- board text added: "-"
- board text added: "160- 180V DC"
- board text added: "5V"
- board text added: "9 - 12V DC"
- board text added: "CS"
- board text added: "Flash"
- board text added: "GND"
- board text added: "HV On"
- board text added: "High Voltage!"
- board text added: "MOSI"
- board text added: "PWM"
- board text added: "Power OK"
- board text added: "RX"
- board text added: "Reset"
- board text added: "SCK"
- board text added: "Sensor"
- board text added: "Status"
- board text added: "TX"

Commit message: Layout done, before PCB order
Parts:
- added G***: LOGO, Loewe:Loewe_Klein, F.Cu at (161.5, 95.2)
- added R25: 68k, Resistors_THT:R_Axial_DIN0207_L6.3mm_D2.5mm_P10.16mm_Horizontal, F.Cu at (177.2, 91.4)
- added R27: 27k, Resistors_THT:R_Axial_DIN0207_L6.3mm_D2.5mm_P10.16mm_Horizontal, F.Cu at (173.4, 81.3)
- added REF**: Symbol_HighVoltage_Type2_CopperTop_VerySmall, MySymbols:Symbol_HighVoltage_Type2_SilkBot_VerySmall, F.Cu at (228.6, 80.3)
- CON1: value BARREL_JACK -> Power
- J2: footprint Socket_Strips:Socket_Strip_Straight_1x06_Pitch2.54mm -> Socket_Strips:Socket_Strip_Straight_1x07_Pitch2.54mm
- R11, R15, R16, R2: value 1R -> 1R37
- RV1: footprint Potentiometers:Potentiometer_Trimmer_Piher_PT-6h_Vertical -> Potentiometers:Potentiometer_Trimmer_Bourns_3296X
- RV2: footprint Potentiometers:Potentiometer_Trimmer_Bourns_PV36W -> Potentiometers:Potentiometer_Trimmer_Bourns_3296X
- moved J2 14.0 mm to (87.4, 93.7), turned to 180 degrees
- moved R19 13.8 mm to (174.8, 74.2), turned to 0 degrees
- moved C6 7.11 mm to (149.1, 103.5)
- moved C7 7.11 mm to (147.8, 90.2)
- moved U1 7.11 mm to (149.7, 97.2)
- moved D5 6.94 mm to (178.8, 69.8), turned to 0 degrees
- moved RV2 5.12 mm to (189.9, 98.4)
- moved REF** 4.60 mm to (172.2, 69.1)
- moved IC2 2.54 mm to (99.1, 86.9)
- moved C12 2.29 mm to (99.1, 81.9), turned to 180 degrees
- moved RV1 2.28 mm to (97.8, 98.4), turned to 90 degrees
- moved D3 2.03 mm to (147.3, 84.3)
- moved R5 2.03 mm to (142.2, 84.3)
- moved R7 1.97 mm to (106.7, 81.9), turned to 270 degrees
- moved R21 1.42 mm to (121.9, 97.8), turned to 180 degrees
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Connections:
- net Net-(D5-Pad2) renamed HV_Status
- J2 pad 1: GND -> +12V
- J2 pad 2: +5V -> Net-(IC2-Pad4)
- J2 pad 3: Net-(IC2-Pad4) -> Net-(IC2-Pad2)
- J2 pad 4: Net-(IC2-Pad3) -> Net-(IC2-Pad5)
- J2 pad 5: Net-(IC2-Pad5) -> Net-(IC2-Pad3)
- J2 pad 6: Net-(IC2-Pad2) -> GND
Routing:
- net GND: track 110.5 -> 471.6 mm, vias 27 -> 89
- net (no net): track 0.00 -> 214.2 mm, vias 0 -> 42
- net +12V: track 138.8 -> 246.1 mm, vias 1 -> 4
- net Net-(R25-Pad1): track 23.0 -> 71.8 mm, vias 0 -> 2
- net +5V: track 118.4 -> 142.6 mm, vias 2 -> 4
- net HV_Status: track 12.0 -> 22.9 mm
- net +3V3: track 88.7 -> 97.2 mm
- net Net-(IC2-Pad4): track 6.98 -> 11.3 mm, vias 1 -> 0
- net Net-(Q5-Pad2): track 42.5 -> 46.2 mm
- net Net-(R4-Pad2): track 6.24 -> 9.51 mm
- net Net-(C14-Pad2): track 28.9 -> 25.7 mm
- net Net-(D5-Pad1): track 4.44 -> 7.03 mm
- net /MOSI: track 11.7 -> 9.13 mm
- net /CS: track 11.1 -> 8.57 mm
- net /PWM: track 12.2 -> 9.69 mm
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Other:
- board text added: "12V"
- board text added: "3V3 OK"
- board text added: "9 - 12V DC Center pos."
- board text added: "Nixie Clock Baseboard"
- board text added: "Sensitivity"
- board text added: "Voltage"
- board text removed: "9 - 12V DC"
- board text removed: "Power OK"

Commit message: Production Version, Firmware Work in Progress
Parts:
- IC2: footprint Housings_SSOP:SSOP-20_5.3x7.2mm_Pitch0.65mm -> Housings_SOIC:SOIC-20W_7.5x12.8mm_Pitch1.27mm
- R1: value 549k -> 560k
- R4: value 3k3 -> 3k65
- RV1: footprint Potentiometers:Potentiometer_Trimmer_Bourns_3296X -> Potentiometers:Potentiometer_Trimmer_Bourns_3296Z
- RV2: value 500R -> 1kR; footprint Potentiometers:Potentiometer_Trimmer_Bourns_3296X -> Potentiometers:Potentiometer_Trimmer_Bourns_3296Z
- moved C12 4.45 mm to (99.1, 77.5)
- moved RV1 1.91 mm to (95.9, 98.4)
- moved IC2 1.71 mm to (97.8, 85.7)
- moved R7 1.27 mm to (106.7, 80.6)
- moved RV2 0.64 mm to (189.2, 98.4)
Connections:
- IC2 pad 6: (no net) -> Net-(IC2-Pad6)
- IC2 pad 7: (no net) -> Net-(IC2-Pad7)
- IC2 pad 8: (no net) -> Net-(IC2-Pad8)
- IC2 pad 9: (no net) -> Net-(IC2-Pad9)
- U2 pad 2: (no net) -> Net-(U2-Pad2)
Routing:
- net (no net): track 214.2 -> 0.00 mm, vias 42 -> 0
- net GND: track 471.6 -> 660.8 mm, vias 89 -> 128
- net +5V: track 142.6 -> 130.1 mm, vias 4 -> 1
- net +12V: track 246.1 -> 249.3 mm
- net Net-(IC2-Pad5): track 9.07 -> 6.11 mm, vias 1 -> 0
- net +3V3: track 97.2 -> 100.1 mm
- net Net-(IC2-Pad3): track 8.81 -> 6.11 mm, vias 1 -> 0
- net /CS: track 8.57 -> 9.86 mm
- net Net-(R7-Pad2): track 4.63 -> 5.88 mm
- net Net-(R8-Pad1): track 10.3 -> 9.28 mm
- net /MOSI: track 9.13 -> 10.2 mm
- net /CLK: track 12.3 -> 11.3 mm
- net /PWM: track 9.69 -> 10.5 mm
- net Prx_Det: track 25.4 -> 24.8 mm
- net Net-(C5-Pad1): track 59.1 -> 59.8 mm
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Other:
- board text added: "12V DC Center pos."
- board text removed: "9 - 12V DC Center pos."
