File: Boards/Baseboard/Baseboard.sch (KiCad schematic (older format))
At the start: 45 parts, among them CON1 BARREL_JACK, IC1 MC34063AP, IC2 74HCT245DW, J1 Serial, J2 Display, P1 HV_Supply, Q1 IRF740, Q2 MPSA55, Q3 BC327, Q4 BC337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

Commit message: Layout chnages
Parts:
- removed P1: HV_Supply, Socket_Strips:Socket_Strip_Straight_1x03_Pitch2.54mm, symbol CONN_01X03
- added J3: HV, Socket_Strips:Socket_Strip_Straight_1x02_Pitch2.54mm, symbol Conn_01x02
- added R11, R15, R16: 1R, Resistors_THT:R_Axial_DIN0207_L6.3mm_D2.5mm_P10.16mm_Horizontal, symbol R
- C1: Feld4 (none) -> Low ESR
- D4: value Time -> Status
- Q3, Q4: footprint TO_SOT_Packages_THT:TO-92_Molded_Narrow -> TO_SOT_Packages_THT:TO-92_Inline_Wide
- R1: Feld4 (none) -> 1% Metal
- R12: value 475k -> 470k
- R13: value 475k -> 1k
- R2: value 0R33 -> 1R
- R4: value 3k32 -> 3k4; Feld4 (none) -> 1% Metal
Connections:
- net labels added: 175V, HV_Off
- net labels removed: HV_EN
- wire segments 143 -> 153
Other:
- note added: "0R25 (1,2A Ipk)"
- moved on the sheet: C1, C10, C12, C9, IC2B, L1, R6, SW1

Commit message: Board layout done
Parts:
- removed C4: 2µ2, Capacitors_THT:CP_Radial_D6.3mm_P2.50mm, symbol CP
- removed Q2: MPSA55, TO_SOT_Packages_THT:TO-92_Inline_Wide, symbol Q_PNP_BCE
- added C13: 100nF, Capacitors_SMD:C_0805_HandSoldering, symbol C
- added C14, C4: 1.5nF, Capacitors_THT:C_Disc_D3.0mm_W2.0mm_P2.50mm, symbol C
- added D5: LED, LEDs:LED_D3.0mm, symbol LED
- added D6: D_TVS, Diodes_THT:D_5W_P12.70mm_Horizontal, symbol D_TVS
- added D7: 1N5711, Diodes_THT:D_DO-35_SOD27_P10.16mm_Horizontal, symbol D
- added D8: ZD20 / 1W, Diodes_THT:D_DO-41_SOD81_P10.16mm_Horizontal, symbol D_Zener
- added J4: Sensor, Measurement_Points:Measurement_Point_Square-TH_Small, symbol Conn_01x01
- added Q2: BC327, TO_SOT_Packages_THT:TO-92_Inline_Wide, symbol BC327
- added Q5: BS170, TO_SOT_Packages_THT:TO-92_Molded_Narrow, symbol BS170
- added Q6, Q8: BC337, TO_SOT_Packages_THT:TO-92_Inline_Wide, symbol BC337
- added Q7: MPSA42, TO_SOT_Packages_THT:TO-92_Molded_Narrow, symbol MPSA42
- added R17: 220k, Resistors_THT:R_Axial_DIN0207_L6.3mm_D2.5mm_P10.16mm_Horizontal, symbol R
- added R18: 120k, Resistors_THT:R_Axial_DIN0207_L6.3mm_D2.5mm_P10.16mm_Horizontal, symbol R
- added R19: 680R, Resistors_THT:R_Axial_DIN0207_L6.3mm_D2.5mm_P10.16mm_Horizontal, symbol R
- added R20, R21: 10k, Resistors_SMD:R_0805_HandSoldering, symbol R
- added R22, R26: 1k, Resistors_THT:R_Axial_DIN0207_L6.3mm_D2.5mm_P10.16mm_Horizontal, symbol R
- added R23: 47R, Resistors_THT:R_Axial_DIN0207_L6.3mm_D2.5mm_P10.16mm_Horizontal, symbol R
- added R24: 4k7, Resistors_THT:R_Axial_DIN0207_L6.3mm_D2.5mm_P10.16mm_Horizontal, symbol R
- added RV1: 100k, Potentiometers:Potentiometer_Trimmer_Piher_PT-6h_Vertical, symbol POT
- added RV2: 500R, Potentiometers:Potentiometer_Trimmer_Bourns_PV36W, symbol POT
- added U4: MTCH101, TO_SOT_Packages_SMD:SOT-23-6_Handsoldering, symbol MTCH101
- C2: Feld4 (none) -> Low ESR
- C5: value 100nF -> 10nF
- D1: value BAV21 -> MUR120; footprint Diodes_THT:D_DO-35_SOD27_P10.16mm_Horizontal -> Diodes_THT:D_DO-15_P10.16mm_Horizontal
- L1: value 220µH -> 270µH / 1.2A; footprint Inductors_THT:L_Radial_D6.0mm_P4.00mm -> Inductors_THT:L_Radial_D12.5mm_P7.00mm_Fastron_09HCP
- R1: value 475k -> 549k
- R10, R5: value R -> 68R
- R11, R15, R16, R2: value 1R -> 1R37
- R12: value 470k -> 4k7
- R13: value 1k -> 180R
- R14: value 4k7 -> 1k
- R4: value 3k4 -> 3k3
- R8: value 470R -> 10k
Connections:
- net +12V: now also D6.1 (A1), Q5.1 (D), R22.2, R24.2; no longer Q3.3 (E)
- net +3V3: now also C13.1, R20.1, R21.1, RV1.1, U4.5 (VDD)
- net 175V: now also D8.1 (K), R17.2
- net GND: now also Q3.1 (C), C13.2, C4.2, D6.2 (A2), Q2.1 (C), Q7.1 (E), Q8.3 (E), R18.1, R19.2, RV1.3, U4.2 (VSS); no longer R8.2
- net at C1.1, IC1.1 (SWC), IC1.7 (IS)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: now also R13.2; no longer IC1.8 (DC)
- net at D2.2 (A), IC1.2 (SWE), R3.2: now also Q3.2 (B)
- net at IC1.3 (TC): now also D7.2 (A), Q2.2 (B)
- net at C5.1, IC1.5 (FB), R1.1: now also Q6.3 (E), RV2.2, RV2.3; no longer Q3.1 (C), R4.2
- net at D2.1 (K), Q1.1 (G): now also Q3.3 (E)
- net at U2.11 (GPIO2): now also R10.1; no longer R8.1
- net Prx_Det: now reaches U2.13 (GPIO5)
- net Prx_Det: now also R21.2, U4.4 (MTO); no longer R10.1
- net at R13.1: now also IC1.8 (DC); no longer Q4.1 (C)
- net HV_Off renamed HV_On
- net HV_On: now also R26.2
- new net: R4.2, RV2.1
- new net: Q4.1 (C), Q6.2 (B), R12.1
- new net: D5.1 (K), R19.1
- new net: D5.2 (A), Q5.3 (S)
- new net: Q5.2 (G), R17.1, R18.2
- new net: J4.1 (Pin_1), U4.1 (MTI)
- new net: R8.1, U4.3 (MTSA)
- new net: R20.2, U4.6 (MTPM)
- new net: R8.2, RV1.2
- new net: C4.1, D7.1 (K), Q2.3 (E)
- new net: Q6.1 (C), R22.1
- new net: C14.1, Q7.3 (C), R23.1
- new net: D8.2 (A), R23.2
- new net: C14.2, Q7.2 (B), Q8.1 (C), R24.1
- new net: Q8.2 (B), R26.1
Other:
- note added: "0R34\n(0,9A Ipk)"
- note added: "Proximity Detector"
- note removed: "0R25 (1,2A Ipk)"
- moved on the sheet: C1, C11, C2, C3, C5, C6, C7, C8, CON1, D1, D2, D3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

Commit message: Layout done, before PCB order
Parts:
- removed J2: Display, Socket_Strips:Socket_Strip_Straight_1x06_Pitch2.54mm, symbol Conn_01x06
- added J2: Display, Socket_Strips:Socket_Strip_Straight_1x07_Pitch2.54mm, symbol Conn_01x07
- added R25: 68k, Resistors_THT:R_Axial_DIN0207_L6.3mm_D2.5mm_P10.16mm_Horizontal, symbol R
- added R27: 27k, Resistors_THT:R_Axial_DIN0207_L6.3mm_D2.5mm_P10.16mm_Horizontal, symbol R
- CON1: value BARREL_JACK -> Power
- R1: value 549k -> 560k
- R4: value 3k3 -> 3k65
- RV1: footprint Potentiometers:Potentiometer_Trimmer_Piher_PT-6h_Vertical -> Potentiometers:Potentiometer_Trimmer_Bourns_3296X
- RV2: value 500R -> 1kR; footprint Potentiometers:Potentiometer_Trimmer_Bourns_PV36W -> Potentiometers:Potentiometer_Trimmer_Bourns_3296X
Connections:
- net +12V: now also J2.1 (Pin_1)
- net +5V: now also J2.7 (Pin_7)
- net GND: now also J2.6 (Pin_6), R27.1
- net at R9.1, U2.12 (GPIO0): now also R25.1, R27.2
- net at IC2.4 (A3): now also J2.2 (Pin_2)
- net at IC2.3 (A2): now also J2.5 (Pin_5)
- net at IC2.5 (A4): now also J2.4 (Pin_4)
- net at IC2.2 (A1): now also J2.3 (Pin_3)
- net HV_Status: now reaches D5.2 (A), Q5.3 (S)
- net HV_Status: now also R25.2
Other:
- moved on the sheet: C13, D5, J4, R18, R19, R20, R21, R8, RV1, U4

Commit message: Production Version, Firmware Work in Progress
Parts:
- C1, C11, C2, C6, C7, C8: symbol CP -> Baseboard-rescue:CP
- C10, C12, C13, C14, C3, C4, C5, C9: symbol C -> Baseboard-rescue:C
- CON1: symbol BARREL_JACK -> Baseboard-rescue:BARREL_JACK
- D1, D2, D7: symbol D -> Baseboard-rescue:D
- D3, D4, D5: symbol LED -> Baseboard-rescue:LED
- D6: symbol D_TVS -> Baseboard-rescue:D_TVS
- D8: symbol D_Zener -> Baseboard-rescue:D_Zener
- IC1: symbol MC34063AP -> Baseboard-rescue:MC34063AP
- IC2: footprint Housings_SSOP:SSOP-20_5.3x7.2mm_Pitch0.65mm -> Housings_SOIC:SOIC-20W_7.5x12.8mm_Pitch1.27mm; symbol 74HCT245DW -> Baseboard-rescue:74HCT245DW
- J1: symbol Conn_01x03 -> Baseboard-rescue:Conn_01x03
- J2: symbol Conn_01x07 -> Baseboard-rescue:Conn_01x07
- J3: symbol Conn_01x02 -> Baseboard-rescue:Conn_01x02
- J4: symbol Conn_01x01 -> Baseboard-rescue:Conn_01x01
- L1: symbol INDUCTOR_SMALL -> Baseboard-rescue:INDUCTOR_SMALL
- Q1: symbol Q_NMOS_GDS -> Baseboard-rescue:Q_NMOS_GDS
- Q2, Q3: symbol BC327 -> Baseboard-rescue:BC327
- Q4, Q6, Q8: symbol BC337 -> Baseboard-rescue:BC337
- Q5: symbol BS170 -> Baseboard-rescue:BS170
- Q7: symbol MPSA42 -> Baseboard-rescue:MPSA42
- R1, R10, R12, R13, R14, R17, R18, R19, R20, R21, R22, R23, R24, R25, R26, R27, R3, R4, R5, R6, R7, R8, R9: symbol R -> Baseboard-rescue:R
- R11, R15, R16, R2: value 1R37 -> 1R; symbol R -> Baseboard-rescue:R
- RV1, RV2: footprint Potentiometers:Potentiometer_Trimmer_Bourns_3296X -> Potentiometers:Potentiometer_Trimmer_Bourns_3296Z; symbol POT -> Baseboard-rescue:POT
- SW1, SW2: symbol SW_Push -> Baseboard-rescue:SW_Push
- U1: symbol LM1117-5.0 -> Baseboard-rescue:LM1117-5.0
- U2: symbol ESP-12 -> Baseboard-rescue:ESP-12
- U3: symbol LM1117-3.3 -> Baseboard-rescue:LM1117-3.3
- U4: symbol MTCH101 -> Baseboard-rescue:MTCH101
Other:
- note added: "3x1R = 0R33\n(0,9A Ipk)\n\n4x1R = 0R25\n(1,2A Ipk)\n\n"
- note added: "Optional"
- note removed: "0R34\n(0,9A Ipk)"
