File: Boards/IN14_Display/IN14_Display.kicad_pcb (KiCad board)
At the start: 2 copper layers, 160 x 50 mm, 49 parts, among them IC1 TPIC6B596DW, IC2 TPIC6B596DW, IC3 TPIC6B596DW, IC4 TPIC6B596DW, IC5 TPIC6B596DW, IC6 TPIC6B596DW, IC7 TPIC6B596DW, IC8 TPIC6B596DW, P1 CONN_01X02, P2 CONN_01X06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

Commit message: Layout chnages
Parts:
- R1, R2, R3, R4, R5, R6: value 22k -> 2k2
- R10, R11, R12, R7, R8, R9: value 270R -> 120R
- R13: value 270R -> 4k7
- R14, R15: value 22k -> 16k
- moved P2 5.44 mm to (68.6, 103.2)
- moved P1 3.57 mm to (218.6, 98.1)
Routing:
- net Net-(P2-Pad3): track 18.9 -> 13.0 mm
- net VCC: track 353.9 -> 357.9 mm
- net Net-(P1-Pad1): track 137.8 -> 141.6 mm
- net Net-(IC1-Pad3): track 9.53 -> 12.3 mm
- net Net-(IC1-Pad13): track 164.3 -> 162.2 mm
- net Net-(IC1-Pad12): track 163.7 -> 162.7 mm
- net Net-(IC8-Pad15): track 17.0 -> 16.1 mm
- net Net-(IC8-Pad14): track 16.7 -> 16.0 mm

Commit message: Board layout done
Parts:
- C1, C2, C3, C4, C5, C6, C7, C8: footprint Capacitors_SMD:C_0805_HandSoldering -> Capacitors_SMD:C_0805
- Q1: value Q_NPN_BCE -> BC817; footprint TO_SOT_Packages_SMD:SOT-23_Handsoldering -> TO_SOT_Packages_SMD:SOT-23
- R10, R11, R12, R7, R8, R9: moved to B.Cu
- R13: value 4k7 -> 2k2
- moved R13 6.52 mm to (75.2, 107.7)
- moved Q1 1.63 mm to (78.7, 107.7), turned to 0 degrees
- moved D6 0.77 mm to (152.4, 107.7)
- moved D1 0.76 mm to (89.8, 107.7)
- moved D2 0.76 mm to (107.3, 107.7)
- moved D3 0.76 mm to (197.3, 107.7)
- moved D4 0.76 mm to (134.7, 107.7)
- moved D5 0.76 mm to (179.8, 107.7)
Connections:
- Q1 pad 2: Net-(D1-Pad1) -> GND
- Q1 pad 3: GND -> Net-(D1-Pad1)
Routing:
- net GND: track 453.8 -> 483.4 mm, vias 126 -> 131
- net Net-(D1-Pad1): track 129.7 -> 134.2 mm
- net Net-(IC6-Pad4): track 34.4 -> 37.9 mm
- net Net-(IC6-Pad5): track 29.4 -> 31.6 mm
- net Net-(D1-Pad2): track 2.69 -> 4.60 mm, vias 0 -> 1
- net Net-(D3-Pad2): track 2.43 -> 4.30 mm, vias 0 -> 1
- net Net-(D5-Pad2): track 2.71 -> 4.38 mm, vias 0 -> 1
- net Net-(D4-Pad2): track 2.66 -> 4.30 mm, vias 0 -> 1
- net Net-(P2-Pad3): track 13.0 -> 11.4 mm
- net Net-(D2-Pad2): track 2.75 -> 4.34 mm, vias 0 -> 1
- net Net-(IC1-Pad5): track 30.5 -> 31.9 mm
- net VCC: track 357.9 -> 356.6 mm, vias 15 -> 9
- net Net-(D6-Pad2): track 2.78 -> 4.13 mm, vias 0 -> 1
- net Net-(IC1-Pad4): track 35.6 -> 36.9 mm
- net Net-(IC1-Pad3): track 12.3 -> 11.1 mm
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
Commit message: Layout done, before PCB order
Parts:
- removed P2: CONN_01X06, Pin_Headers:Pin_Header_Straight_1x06_Pitch2.54mm
- removed the REF** at (216.5, 110.5)
- added J1: Conn_01x07, Pin_Headers:Pin_Header_Straight_1x07_Pitch2.54mm, B.Cu at (68.8, 104.5)
- added R16: 16k, Resistors_SMD:R_0805, F.Cu at (214.4, 99.3)
- added REF**: Symbol_HighVoltage_Type2_CopperTop_VerySmall, MySymbols:Symbol_HighVoltage_Type2_SilkTop_VerySmall, F.Cu at (217.4, 105.2)
- C1, C2, C3, C4, C5, C6, C7, C8: moved to F.Cu
- moved C2 96.0 mm to (92.7, 82.3)
- moved C7 66.5 mm to (182.6, 82.3)
- moved R9 64.5 mm to (133.1, 109.2), turned to 90 degrees
- moved D3 64.0 mm to (133.3, 108.4)
- moved C4 48.8 mm to (128.5, 82.3)
- moved D6 46.4 mm to (198.8, 108.4)
- moved R12 46.3 mm to (198.9, 109.2), turned to 90 degrees
- moved C3 24.5 mm to (110.5, 82.3)
- moved C1 24.1 mm to (74.7, 82.3)
- moved C5 24.0 mm to (146.6, 82.3)
- moved D4 19.1 mm to (153.8, 108.4)
- moved R10 19.0 mm to (153.7, 109.2), turned to 90 degrees
- moved R2 18.8 mm to (108.7, 98.7), turned to 270 degrees
- moved R5 18.8 mm to (178.3, 98.7), turned to 270 degrees
- moved R4 18.8 mm to (153.8, 98.7), turned to 270 degrees
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Connections:
- IC1 pad 10: (no net) -> GND
- IC1 pad 11: (no net) -> GND
- IC1 pad 18: Net-(IC1-Pad18) -> (no net)
- IC1 pad 19: (no net) -> GND
- IC1 pad 2: (no net) -> VCC
- IC2 pad 10: (no net) -> GND
- IC2 pad 11: (no net) -> GND
- IC2 pad 18: Net-(IC2-Pad18) -> Net-(IC1-Pad3)
- IC2 pad 19: (no net) -> GND
- IC2 pad 2: (no net) -> VCC
- IC2 pad 3: Net-(IC1-Pad18) -> Net-(IC2-Pad3)
- IC3 pad 10: (no net) -> GND
- IC3 pad 11: (no net) -> GND
- IC3 pad 18: Net-(IC3-Pad18) -> Net-(IC2-Pad3)
- IC3 pad 19: (no net) -> GND
- IC3 pad 2: (no net) -> VCC
- IC3 pad 3: Net-(IC2-Pad18) -> Net-(IC3-Pad3)
- IC4 pad 10: (no net) -> GND
- IC4 pad 11: (no net) -> GND
- IC4 pad 18: Net-(IC4-Pad18) -> Net-(IC3-Pad3)
- IC4 pad 19: (no net) -> GND
- IC4 pad 2: (no net) -> VCC
- IC4 pad 3: Net-(IC3-Pad18) -> Net-(IC4-Pad3)
- IC5 pad 10: (no net) -> GND
- IC5 pad 11: (no net) -> GND
- IC5 pad 18: Net-(IC5-Pad18) -> Net-(IC4-Pad3)
- IC5 pad 19: (no net) -> GND
- IC5 pad 2: (no net) -> VCC
- IC5 pad 3: Net-(IC4-Pad18) -> Net-(IC5-Pad3)
- IC6 pad 10: (no net) -> GND
- IC6 pad 11: (no net) -> GND
- IC6 pad 18: Net-(IC6-Pad18) -> Net-(IC5-Pad3)
- IC6 pad 19: (no net) -> GND
- IC6 pad 2: (no net) -> VCC
- IC6 pad 3: Net-(IC5-Pad18) -> Net-(IC6-Pad3)
- IC7 pad 10: (no net) -> GND
- IC7 pad 11: (no net) -> GND
- IC7 pad 18: Net-(IC7-Pad18) -> Net-(IC6-Pad3)
- IC7 pad 19: (no net) -> GND
- IC7 pad 2: (no net) -> VCC
- IC7 pad 3: Net-(IC6-Pad18) -> Net-(IC7-Pad3)
- IC8 pad 10: (no net) -> GND
- IC8 pad 11: (no net) -> GND
- IC8 pad 16: (no net) -> Net-(IC8-Pad16)
- IC8 pad 18: (no net) -> Net-(IC7-Pad3)
- IC8 pad 19: (no net) -> GND
- IC8 pad 2: (no net) -> VCC
- IC8 pad 3: Net-(IC7-Pad18) -> Net-(IC8-Pad3)
- N2 pad RHDP: (no net) -> Net-(N2-PadRHDP)
- N4 pad RHDP: (no net) -> Net-(N4-PadRHDP)
- N6 pad LHDP: Net-(N6-PadLHDP) -> (no net)
- R10 pad 1: VCC -> +12V
- R11 pad 1: VCC -> +12V
- R12 pad 1: VCC -> +12V
- R14 pad 1: Net-(N6-PadLHDP) -> Net-(IC8-Pad15)
- R14 pad 2: Net-(IC8-Pad14) -> Net-(N4-PadRHDP)
- R15 pad 1: Net-(N6-PadRHDP) -> Net-(IC8-Pad14)
- R15 pad 2: Net-(IC8-Pad15) -> Net-(N6-PadRHDP)
- R7 pad 1: VCC -> +12V
- R8 pad 1: VCC -> +12V
- R9 pad 1: VCC -> +12V
Routing:
- net Net-(IC8-Pad3): track 0.00 -> 148.8 mm, vias 0 -> 1
- net +12V: track 0.00 -> 136.4 mm
- net Net-(N2-PadRHDP): track 0.00 -> 130.7 mm, vias 0 -> 1
- net GND: track 483.4 -> 613.4 mm, vias 131 -> 115
- net VCC: track 356.6 -> 273.7 mm, vias 9 -> 15
- net Net-(N4-PadRHDP): track 0.00 -> 79.2 mm, vias 0 -> 1
- net Net-(IC6-Pad3): track 0.00 -> 34.6 mm, vias 0 -> 2
- net Net-(IC4-Pad3): track 0.00 -> 34.2 mm, vias 0 -> 2
- net Net-(IC3-Pad7): track 27.7 -> 61.2 mm
- net Net-(IC2-Pad3): track 0.00 -> 33.4 mm, vias 0 -> 2
- net Net-(IC8-Pad7): track 28.1 -> 61.4 mm
- net Net-(IC8-Pad6): track 25.2 -> 57.8 mm
- net Net-(IC3-Pad6): track 24.8 -> 57.4 mm
- net Net-(IC3-Pad3): track 0.00 -> 31.9 mm, vias 0 -> 2
- net Net-(IC7-Pad3): track 0.00 -> 31.4 mm, vias 0 -> 2
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Other:
- board text added: "D. Walter v1.0"
- board text added: "IN14 Display Board"

Commit message: Production Version, Firmware Work in Progress
Connections:
- IC1 pad 18: (no net) -> Net-(IC1-Pad18)
- IC8 pad 17: (no net) -> Net-(IC8-Pad17)
- J1 pad 6: VCC -> GND
- J1 pad 7: GND -> VCC
- N1 pad LHDP: (no net) -> Net-(N1-PadLHDP)
- N1 pad RHDP: (no net) -> Net-(N1-PadRHDP)
- N2 pad LHDP: (no net) -> Net-(N2-PadLHDP)
- N3 pad LHDP: (no net) -> Net-(N3-PadLHDP)
- N3 pad RHDP: (no net) -> Net-(N3-PadRHDP)
- N4 pad LHDP: (no net) -> Net-(N4-PadLHDP)
- N5 pad LHDP: (no net) -> Net-(N5-PadLHDP)
- N5 pad RHDP: (no net) -> Net-(N5-PadRHDP)
- N6 pad LHDP: (no net) -> Net-(N6-PadLHDP)
Routing:
- net GND: track 613.4 -> 610.5 mm
- net VCC: track 273.7 -> 272.4 mm
- net Net-(IC5-Pad14): track 41.4 -> 42.1 mm
- net Net-(IC5-Pad15): track 47.5 -> 48.2 mm
- net Net-(IC5-Pad16): track 54.1 -> 54.7 mm
- net Net-(IC5-Pad17): track 61.0 -> 61.5 mm
- net Net-(IC5-Pad7): track 48.7 -> 49.2 mm
Other:
- board text added: "D. Walter v1.1"
- board text removed: "D. Walter v1.0"
