File: Boards/IN14_Display/IN14_Display.sch (KiCad schematic (older format))
At the start: 46 parts, among them IC1 TPIC6B596DW, IC2 TPIC6B596DW, IC3 TPIC6B596DW, IC4 TPIC6B596DW, IC5 TPIC6B596DW, IC6 TPIC6B596DW, IC7 TPIC6B596DW, IC8 TPIC6B596DW, P1 CONN_01X02, P2 CONN_01X06, Q1 Q_NPN_BCE

Commit message: Layout chnages
Parts:
- R1, R2, R3, R4, R5, R6: value 22k -> 2k2
- R10, R11, R12, R7, R8, R9: value 270R -> 120R
- R13: value 270R -> 4k7
- R14, R15: value 22k -> 16k
Changed lines of the file:
@@
 P 1650 6150
 F 0 "R7" V 1730 6150 50  0000 C CNN
-F 1 "270R" V 1650 6150 50  0000 C CNN
+F 1 "120R" V 1650 6150 50  0000 C CNN
 F 2 "Resistors_SMD:R_0805" V 1580 6150 50  0001 C CNN
 F 3 "" H 1650 6150 50  0000 C CNN
@@
 P 1550 1750
 F 0 "R1" V 1630 1750 50  0000 C CNN
-F 1 "22k" V 1550 1750 50  0000 C CNN
+F 1 "2k2" V 1550 1750 50  0000 C CNN
 F 2 "Resistors_SMD:R_0805" V 1480 1750 50  0001 C CNN
 F 3 "" H 1550 1750 50  0000 C CNN
@@
 P 3100 1750
 F 0 "R2" V 3180 1750 50  0000 C CNN
-F 1 "22k" V 3100 1750 50  0000 C CNN
+F 1 "2k2" V 3100 1750 50  0000 C CNN
 F 2 "Resistors_SMD:R_0805" V 3030 1750 50  0001 C CNN
 F 3 "" H 3100 1750 50  0000 C CNN
@@
 P 4650 1750
 F 0 "R3" V 4730 1750 50  0000 C CNN
-F 1 "22k" V 4650 1750 50  0000 C CNN
+F 1 "2k2" V 4650 1750 50  0000 C CNN
 F 2 "Resistors_SMD:R_0805" V 4580 1750 50  0001 C CNN
 F 3 "" H 4650 1750 50  0000 C CNN
@@
 P 6200 1750
 F 0 "R4" V 6280 1750 50  0000 C CNN
-F 1 "22k" V 6200 1750 50  0000 C CNN
+F 1 "2k2" V 6200 1750 50  0000 C CNN
 F 2 "Resistors_SMD:R_0805" V 6130 1750 50  0001 C CNN
 F 3 "" H 6200 1750 50  0000 C CNN
@@
 P 8200 1750
 F 0 "R5" V 8280 1750 50  0000 C CNN
-F 1 "22k" V 8200 1750 50  0000 C CNN
+F 1 "2k2" V 8200 1750 50  0000 C CNN
 F 2 "Resistors_SMD:R_0805" V 8130 1750 50  0001 C CNN
 F 3 "" H 8200 1750 50  0000 C CNN
@@
 P 9700 1750
 F 0 "R6" V 9780 1750 50  0000 C CNN
-F 1 "22k" V 9700 1750 50  0000 C CNN
+F 1 "2k2" V 9700 1750 50  0000 C CNN
 F 2 "Resistors_SMD:R_0805" V 9630 1750 50  0001 C CNN
 F 3 "" H 9700 1750 50  0000 C CNN
@@
 P 1950 6150
 F 0 "R8" V 2030 6150 50  0000 C CNN
-F 1 "270R" V 1950 6150 50  0000 C CNN
+F 1 "120R" V 1950 6150 50  0000 C CNN
 F 2 "Resistors_SMD:R_0805" V 1880 6150 50  0001 C CNN
 F 3 "" H 1950 6150 50  0000 C CNN
@@
 P 2250 6150
 F 0 "R9" V 2330 6150 50  0000 C CNN
-F 1 "270R" V 2250 6150 50  0000 C CNN
+F 1 "120R" V 2250 6150 50  0000 C CNN
 F 2 "Resistors_SMD:R_0805" V 2180 6150 50  0001 C CNN
 F 3 "" H 2250 6150 50  0000 C CNN
@@
 P 2550 6150
 F 0 "R10" V 2630 6150 50  0000 C CNN
-F 1 "270R" V 2550 6150 50  0000 C CNN
+F 1 "120R" V 2550 6150 50  0000 C CNN
 F 2 "Resistors_SMD:R_0805" V 2480 6150 50  0001 C CNN
 F 3 "" H 2550 6150 50  0000 C CNN
@@
 P 2850 6150
 F 0 "R11" V 2930 6150 50  0000 C CNN
-F 1 "270R" V 2850 6150 50  0000 C CNN
+F 1 "120R" V 2850 6150 50  0000 C CNN
 F 2 "Resistors_SMD:R_0805" V 2780 6150 50  0001 C CNN
 F 3 "" H 2850 6150 50  0000 C CNN
@@
 P 3150 6150
 F 0 "R12" V 3230 6150 50  0000 C CNN
-F 1 "270R" V 3150 6150 50  0000 C CNN
+F 1 "120R" V 3150 6150 50  0000 C CNN
 F 2 "Resistors_SMD:R_0805" V 3080 6150 50  0001 C CNN
 F 3 "" H 3150 6150 50  0000 C CNN
@@
 P 1800 7000
 F 0 "R13" V 1880 7000 50  0000 C CNN
-F 1 "270R" V 1800 7000 50  0000 C CNN
+F 1 "4k7" V 1800 7000 50  0000 C CNN
 F 2 "Resistors_SMD:R_0805" V 1730 7000 50  0001 C CNN
 F 3 "" H 1800 7000 50  0000 C CNN
@@
 P 10800 2250
 F 0 "R15" V 10880 2250 50  0000 C CNN
-F 1 "22k" V 10800 2250 50  0000 C CNN
+F 1 "16k" V 10800 2250 50  0000 C CNN
 F 2 "Resistors_SMD:R_0805" V 10730 2250 50  0001 C CNN
 F 3 "" H 10800 2250 50  0000 C CNN
@@
 P 10700 1600
 F 0 "R14" V 10780 1600 50  0000 C CNN
-F 1 "22k" V 10700 1600 50  0000 C CNN
+F 1 "16k" V 10700 1600 50  0000 C CNN
 F 2 "Resistors_SMD:R_0805" V 10630 1600 50  0001 C CNN
 F 3 "" H 10700 1600 50  0000 C CNN

Commit message: Board layout done
Parts:
- removed Q1: Q_NPN_BCE, TO_SOT_Packages_SMD:SOT-23_Handsoldering, symbol Q_NPN_BCE
- added Q1: BC817, TO_SOT_Packages_SMD:SOT-23, symbol BC817
- C1, C2, C3, C4, C5, C6, C7, C8: footprint Capacitors_SMD:C_0805_HandSoldering -> Capacitors_SMD:C_0805
- R13: value 4k7 -> 2k2
Connections:
- net GND: now also Q1.2 (E)
- net at D1.1 (K), D2.1 (K), D3.1 (K)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: now also Q1.3 (C)
- net at R13.1: now also Q1.1 (B)
Changed lines of the file:
@@
 F 0 "C1" H 3725 6300 50  0000 L CNN
 F 1 "100nF" H 3725 6100 50  0000 L CNN
-F 2 "Capacitors_SMD:C_0805_HandSoldering" H 3738 6050 50  0001 C CNN
+F 2 "Capacitors_SMD:C_0805" H 3738 6050 50  0001 C CNN
 F 3 "" H 3700 6200 50  0000 C CNN
 	1    3700 6200
@@
 F 0 "C2" H 4075 6300 50  0000 L CNN
 F 1 "100nF" H 4075 6100 50  0000 L CNN
-F 2 "Capacitors_SMD:C_0805_HandSoldering" H 4088 6050 50  0001 C CNN
+F 2 "Capacitors_SMD:C_0805" H 4088 6050 50  0001 C CNN
 F 3 "" H 4050 6200 50  0000 C CNN
 	1    4050 6200
@@
 F 0 "C3" H 4425 6300 50  0000 L CNN
 F 1 "100nF" H 4425 6100 50  0000 L CNN
-F 2 "Capacitors_SMD:C_0805_HandSoldering" H 4438 6050 50  0001 C CNN
+F 2 "Capacitors_SMD:C_0805" H 4438 6050 50  0001 C CNN
 F 3 "" H 4400 6200 50  0000 C CNN
 	1    4400 6200
@@
 F 0 "C4" H 4775 6300 50  0000 L CNN
 F 1 "100nF" H 4775 6100 50  0000 L CNN
-F 2 "Capacitors_SMD:C_0805_HandSoldering" H 4788 6050 50  0001 C CNN
+F 2 "Capacitors_SMD:C_0805" H 4788 6050 50  0001 C CNN
 F 3 "" H 4750 6200 50  0000 C CNN
 	1    4750 6200
@@
 F 0 "C5" H 5125 6300 50  0000 L CNN
 F 1 "100nF" H 5125 6100 50  0000 L CNN
-F 2 "Capacitors_SMD:C_0805_HandSoldering" H 5138 6050 50  0001 C CNN
+F 2 "Capacitors_SMD:C_0805" H 5138 6050 50  0001 C CNN
 F 3 "" H 5100 6200 50  0000 C CNN
 	1    5100 6200
@@
 F 0 "C6" H 5475 6300 50  0000 L CNN
 F 1 "100nF" H 5475 6100 50  0000 L CNN
-F 2 "Capacitors_SMD:C_0805_HandSoldering" H 5488 6050 50  0001 C CNN
+F 2 "Capacitors_SMD:C_0805" H 5488 6050 50  0001 C CNN
 F 3 "" H 5450 6200 50  0000 C CNN
 	1    5450 6200
@@
 F 0 "C7" H 5825 6300 50  0000 L CNN
 F 1 "100nF" H 5825 6100 50  0000 L CNN
-F 2 "Capacitors_SMD:C_0805_HandSoldering" H 5838 6050 50  0001 C CNN
+F 2 "Capacitors_SMD:C_0805" H 5838 6050 50  0001 C CNN
 F 3 "" H 5800 6200 50  0000 C CNN
 	1    5800 6200
@@
 $EndComp
 $Comp
-L Q_NPN_BCE Q1
-U 1 1 587057EA
-P 2300 7000
-F 0 "Q1" H 2500 7050 50  0000 L CNN
-F 1 "Q_NPN_BCE" H 2500 6950 50  0000 L CNN
-F 2 "TO_SOT_Packages_SMD:SOT-23_Handsoldering" H 2500 7100 50  0001 C CNN
-F 3 "" H 2300 7000 50  0000 C CNN
-	1    2300 7000
-	1    0    0    -1
-$EndComp
-$Comp
 L LED D2
 U 1 1 5870646E
@@
 P 1800 7000
 F 0 "R13" V 1880 7000 50  0000 C CNN
-F 1 "4k7" V 1800 7000 50  0000 C CNN
+F 1 "2k2" V 1800 7000 50  0000 C CNN
 F 2 "Resistors_SMD:R_0805" V 1730 7000 50  0001 C CNN
 F 3 "" H 1800 7000 50  0000 C CNN
@@
 F 0 "C8" H 6125 6300 50  0000 L CNN
 F 1 "100nF" H 6125 6100 50  0000 L CNN
-F 2 "Capacitors_SMD:C_0805_HandSoldering" H 6138 6050 50  0001 C CNN
+F 2 "Capacitors_SMD:C_0805" H 6138 6050 50  0001 C CNN
 F 3 "" H 6100 6200 50  0000 C CNN
 	1    6100 6200
@@
 	6100 5950 6100 6050
 Connection ~ 5800 5950
+$Comp
+L BC817 Q1
+U 1 1 5A936BEA
+P 2300 7000
+F 0 "Q1" H 2500 7075 50  0000 L CNN
+F 1 "BC817" H 2500 7000 50  0000 L CNN
+F 2 "TO_SOT_Packages_SMD:SOT-23" H 2500 6925 50  0001 L CIN
+F 3 "" H 2300 7000 50  0001 L CNN
+	1    2300 7000
+	1    0    0    -1
+$EndComp
 $EndSCHEMATC

Commit message: Layout done, before PCB order
Parts:
- removed P2: CONN_01X06, Pin_Headers:Pin_Header_Straight_1x06_Pitch2.54mm, symbol CONN_01X06
- added unit 2 of IC1
- added unit 2 of IC2
- added unit 2 of IC3
- added unit 2 of IC4
- added unit 2 of IC5
- added unit 2 of IC6
- added unit 2 of IC7
- added unit 2 of IC8
- added J1: Conn_01x07, Pin_Headers:Pin_Header_Straight_1x07_Pitch2.54mm, symbol Conn_01x07
- added R16: 16k, Resistors_SMD:R_0805, symbol R
Connections:
- net GND: now also IC1.10 (GND@2), IC1.11 (GND@3), IC1.19 (GND@1), IC2.10 (GND@2), IC2.11 (GND@3), IC2.19 (GND@1), IC3.10 (GND@2), IC3.11 (GND@3), IC3.19 (GND@1), IC4.10 (GND@2), IC4.11 (GND@3), IC4.19 (GND@1), IC5.10 (GND@2), IC5.11 (GND@3), IC5.19 (GND@1), IC6.10 (GND@2), IC6.11 (GND@3), IC6.19 (GND@1), IC7.10 (GND@2), IC7.11 (GND@3), IC7.19 (GND@1), IC8.10 (GND@2), IC8.11 (GND@3), IC8.19 (GND@1), J1.7 (Pin_7)
- net VCC: now also IC1.2 (VCC), IC2.2 (VCC), IC3.2 (VCC), IC4.2 (VCC), IC5.2 (VCC), IC6.2 (VCC), IC7.2 (VCC), IC8.2 (VCC), J1.6 (Pin_6); no longer R10.1, R11.1, R12.1, R7.1, R8.1, R9.1
- net at N2.RHDP: now also R16.2
- net at N4.RHDP: now also R14.2
- net at N6.LHDP: no longer R14.1
- net at N6.RHDP: now also R15.2; no longer R15.1
- net at R13.2: now also J1.2 (Pin_2)
- net at IC1.12 (RCK), IC2.12 (RCK), IC3.12 (RCK)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: now also J1.3 (Pin_3)
- net at IC1.13 (SCK), IC2.13 (SCK), IC3.13 (SCK)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: now also J1.4 (Pin_4)
- net at IC1.3 (DI): now also IC2.18 (DO)
- net at IC1.18 (DO): no longer IC2.3 (DI)
- net at IC3.3 (DI): now also IC4.18 (DO); no longer IC2.18 (DO)
- net at IC3.18 (DO): now also IC2.3 (DI); no longer IC4.3 (DI)
- net at IC5.3 (DI): now also IC6.18 (DO); no longer IC4.18 (DO)
- net at IC5.18 (DO): now also IC4.3 (DI); no longer IC6.3 (DI)
- net at IC7.3 (DI): now also IC8.18 (DO); no longer IC6.18 (DO)
- net at IC7.18 (DO): now also IC6.3 (DI); no longer IC8.3 (DI)
- net at IC8.14 (Q4): now also R15.1; no longer R14.2
- net at IC8.15 (Q5): now also R14.1; no longer R15.2
- net at IC8.16 (Q6): now also R16.1
- new net: IC8.3 (DI), J1.5 (Pin_5)
- new net +12V: J1.1 (Pin_1), R10.1, R11.1, R12.1, R7.1, R8.1, R9.1
- no-connect marks 13 -> 11
Other:
- moved on the sheet: C1, C2, C3, C4, C5, C6, C7, C8, D1, D2, D3, D4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

Commit message: Production Version, Firmware Work in Progress
Parts:
- C1, C2, C3, C4, C5, C6, C7, C8: symbol C -> Device:C
- D1, D2, D3, D4, D5, D6: symbol LED -> Device:LED
- IC1, IC2, IC3, IC4, IC5, IC6, IC7, IC8: symbol TPIC6B596DW -> tpic:TPIC6B596DW
- J1: symbol Conn_01x07 -> IN14_Display-rescue:Conn_01x07
- N1, N2, N3, N4, N5, N6: symbol IN-14 -> russian-nixies:IN-14
- P1: symbol CONN_01X02 -> IN14_Display-rescue:CONN_01X02
- Q1: symbol BC817 -> IN14_Display-rescue:BC817
- R1, R10, R11, R12, R13, R14, R15, R16, R2, R3, R4, R5, R6, R7, R8, R9: symbol R -> Device:R
Connections:
- net GND: now also J1.6 (Pin_6); no longer J1.7 (Pin_7)
- net VCC: now also J1.7 (Pin_7); no longer J1.6 (Pin_6)
Other:
- moved on the sheet: J1
